File: Hardware/EDA/ESPBee.kicad_pcb (KiCad board)
At the start: 2 copper layers, 24.4 x 27.6 mm, 12 parts, among them P1 XBEE HEADER, P2 HEADER_M_XBEE_P11-P20_PTH_DTE, U1 ESP-12E

Commit message: Added pinout diagram to repository
Parts:
- added SW1: EVQP7A, Electromechanical:EVQP7A, B.Cu at (106.5, 103.0)
- added SW2: EVQP7A, Electromechanical:EVQP7A, B.Cu at (113.0, 103.0)
- moved G1 11.1 mm to (114.5, 93.5)
- moved R4 0.51 mm to (109.5, 98.7)
- moved R2 0.25 mm to (109.5, 96.9)
Routing:
- net GND: track 41.4 -> 56.0 mm
- net /~BOOTLOAD: track 10.0 -> 20.4 mm
- net RST: track 34.1 -> 31.3 mm
- net CTS: track 20.4 -> 23.0 mm
- net VDD: track 31.0 -> 32.6 mm, vias 1 -> 2
Other:
- board text added: "BOOT"
- board text added: "BOOT/"
- board text added: "REV 2.0"
- board text added: "RST"
- board text added: "RST/"
- board text removed: "REV 1.0"
