File: Hardware/EDA/ESPBee.kicad_pcb (KiCad board)
At the start: 2 copper layers, 24.4 x 27.6 mm, 12 parts, among them P1 XBEE HEADER, P2 HEADER_M_XBEE_P11-P20_PTH_DTE, U1 ESP-12E

Commit message: Added test points for Boot and Reset signals. Cleaned up routing.
Parts:
- added TP1: TEST, Wire_to_Board:WIRE_PAD_22AWG, F.Cu at (103.3, 103.7)
- added TP2: TEST, Wire_to_Board:WIRE_PAD_22AWG, F.Cu at (119.1, 103.7)
Connections:
- P1 pad 4: (no net) -> Net-(P1-Pad4)
- P1 pad 6: (no net) -> Net-(P1-Pad6)
- P1 pad 7: (no net) -> Net-(P1-Pad7)
- P1 pad 8: (no net) -> Net-(P1-Pad8)
- P1 pad 9: (no net) -> Net-(P1-Pad9)
- P2 pad 11: (no net) -> Net-(P2-Pad11)
- P2 pad 14: (no net) -> Net-(P2-Pad14)
- P2 pad 15: (no net) -> Net-(P2-Pad15)
- P2 pad 17: (no net) -> Net-(P2-Pad17)
- P2 pad 18: (no net) -> Net-(P2-Pad18)
- P2 pad 19: (no net) -> Net-(P2-Pad19)
- P2 pad 20: (no net) -> Net-(P2-Pad20)
- U1 pad 10: (no net) -> Net-(U1-Pad10)
- U1 pad 11: (no net) -> Net-(U1-Pad11)
- U1 pad 12: (no net) -> Net-(U1-Pad12)
- U1 pad 13: (no net) -> Net-(U1-Pad13)
- U1 pad 14: (no net) -> Net-(U1-Pad14)
- U1 pad 19: (no net) -> Net-(U1-Pad19)
- U1 pad 2: (no net) -> Net-(U1-Pad2)
- U1 pad 20: (no net) -> Net-(U1-Pad20)
- U1 pad 4: (no net) -> Net-(U1-Pad4)
- U1 pad 5: (no net) -> Net-(U1-Pad5)
- U1 pad 6: (no net) -> Net-(U1-Pad6)
- U1 pad 9: (no net) -> Net-(U1-Pad9)
Routing:
- net /~BOOTLOAD: track 10.0 -> 20.8 mm, vias 1 -> 3
- net RST: track 34.1 -> 41.9 mm
- net GND: track 41.4 -> 38.9 mm
- net ON/~SLEEP: track 29.0 -> 27.0 mm
Other:
- board text added: "BOOT"
- board text added: "REV 1.1"
- board text added: "RST"
- board text removed: "REV 1.0"
