File: Hardware/EDA/ESPBee.sch (KiCad schematic (older format))
At the start: 12 parts, among them P1 XBEE HEADER, P2 HEADER_M_XBEE_P11-P20_PTH_DTE, U1 ESP-12E

Commit message: Added pinout diagram to repository
Parts:
- added SW1, SW2: EVQP7A, Electromechanical:EVQP7A, symbol SWITCH_EVQP7A
Connections:
- wire segments 38 -> 46
Other:
- moved on the sheet: R2, R4
