File: Hardware/EDA/ESPBee.sch (KiCad schematic (older format))
At the start: 12 parts, among them P1 XBEE HEADER, P2 HEADER_M_XBEE_P11-P20_PTH_DTE, U1 ESP-12E

Commit message: Added test points for Boot and Reset signals. Cleaned up routing.
Parts:
- added TP1, TP2: TEST, Wire_to_Board:WIRE_PAD_22AWG, symbol TEST
Connections:
- net RST: now also TP1.1
- net ~BOOTLOAD: now also TP2.1
Changed lines of the file:
@@
 LIBS:Mounting_Hole
 LIBS:Transducer
+LIBS:ESPBee-cache
 EELAYER 25 0
 EELAYER END
@@
 Sheet 1 1
 Title "ESPBee"
-Date "2017-07-30"
-Rev "1.0"
+Date "2018-02-16"
+Rev "1.1"
 Comp ""
 Comment1 ""
@@
 	1    0    0    -1
 $EndComp
-Text GLabel 4400 1450 0    40   Input ~ 0
+Text GLabel 4200 1450 0    40   Input ~ 0
 RST
 Wire Wire Line
-	4400 1450 4750 1450
+	4200 1450 4750 1450
 Text GLabel 6050 1550 2    40   Input ~ 0
 RXD
@@
 ~RECOVERY
 NoConn ~ 4800 4550
+$Comp
+L TEST TP1
+U 1 1 5A87D1DE
+P 4300 1350
+F 0 "TP1" H 4300 1550 40  0000 C BNN
+F 1 "TEST" H 4300 1600 40  0001 C CNN
+F 2 "Wire_to_Board:WIRE_PAD_22AWG" H 4300 1350 50  0001 C CNN
+F 3 "" H 4300 1350 50  0001 C CNN
+	1    4300 1350
+	1    0    0    -1
+$EndComp
+$Comp
+L TEST TP2
+U 1 1 5A87D2A4
+P 6550 1750
+F 0 "TP2" H 6550 1950 40  0000 C BNN
+F 1 "TEST" H 6550 2000 50  0001 C CNN
+F 2 "Wire_to_Board:WIRE_PAD_22AWG" H 6550 1750 50  0001 C CNN
+F 3 "" H 6550 1750 50  0001 C CNN
+	1    6550 1750
+	1    0    0    -1
+$EndComp
+Wire Wire Line
+	6550 1750 6550 1850
+Connection ~ 6550 1850
+Wire Wire Line
+	4300 1350 4300 1450
+Connection ~ 4300 1450
 $EndSCHEMATC

Commit message: Updated schematic per remapped schematic decals in KiCAD version 5.0.0.
Signed-off-by: clintastevenson@gmail.com <clintastevenson@gmail.com>
Parts:
- C1, C2, C3, C4: symbol CAP -> Passive:CAP
- G1: symbol Casco_Logix_Logo -> CascoLogixLogo:Casco_Logix_Logo
- P1: symbol HEADER_M_XBEE_P1-P10_PTH_DTE -> Header:HEADER_M_XBEE_P1-P10_PTH_DTE
- P2: symbol HEADER_M_XBEE_P11-P20_PTH_DTE -> Header:HEADER_M_XBEE_P11-P20_PTH_DTE
- R1, R2, R3, R4: symbol RES_Small -> Passive:RES_Small
- TP1, TP2: symbol TEST -> ESPBee-rescue:TEST
- U1: symbol ESP-12E -> RF_Modules:ESP-12E
